File: boards/drive/atlas_drive_i_out.kicad_sch (KiCad schematic)
At the start: 31 parts, among them J901 SERVO, J902 LIDAR_PWR, J903 FAN, U901 TPSM63610, U902 TPS26600

Commit message: Review fixes: docs, run_kicad.sh and drive board text
- README, docs/ARCHITECTURE.md, share/README.md, boards/tools/README.md: status,
  rebuild steps and tool notes brought up to date
- run_kicad.sh: the optional first argument is a sync tarball or an empty string
- Drive schematic text: header J702, 7.5 V servo rail, the precharge resistors
  take 0.15 J each (R319/R320 descriptions synced on the board)
- BOM wording: 7.5 V servo rail

DRC unchanged: no unconnected items, no clearance errors, 8 silkscreen and
track-end warnings.

Co-Authored-By: Claude Opus 5.5 <noreply@anthropic.com>
Claude-Session: https://claude.ai/code/session_01XVBHou86msuHYBGRPr641F
Other:
- note added: "Servo 7.5 V (TPSM63610), lidar eFuse (TPS26600), fan"
- note removed: "Servo 7.4 V (TPSM63610), lidar eFuse (TPS26600), fan"
- title: ATLAS-DRV-1 drive board: Servo 7.4 V (TPSM63610), lidar eFuse (TPS26600), fan -> ATLAS-DRV-1 drive board: Servo 7.5 V (TPSM63610), lidar eFuse (TPS26600), fan
Changed lines of the file:
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@@
 (kicad_sch (version 20250114) (generator "eeschema") (generator_version "9.0")
  (paper "A2")
- (title_block (title "ATLAS-DRV-1 drive board: Servo 7.4 V (TPSM63610), lidar eFuse (TPS26600), fan") (date "2026-09-27") (rev "0.1") (company "Atlas Autoware (501c3), Fairfax VA") (comment 1 "Generated from design.py by tools/eda.py; edit the Python, not this file"))
- (text "Servo 7.4 V (TPSM63610), lidar eFuse (TPS26600), fan" (exclude_from_sim no) (at 25.4 25.4 0) (effects (font (size 3 3) (thickness 0.5) bold) (justify left)))
+ (title_block (title "ATLAS-DRV-1 drive board: Servo 7.5 V (TPSM63610), lidar eFuse (TPS26600), fan") (date "2026-09-27") (rev "0.1") (company "Atlas Autoware (501c3), Fairfax VA") (comment 1 "Generated from design.py by tools/eda.py; edit the Python, not this file"))
+ (text "Servo 7.5 V (TPSM63610), lidar eFuse (TPS26600), fan" (exclude_from_sim no) (at 25.4 25.4 0) (effects (font (size 3 3) (thickness 0.5) bold) (justify left)))
 (text "TPSM63610 from VM: RFBT 100k / RFBB 15.4k = 7.49 V, RT 15.8k = 1 MHz, EN divider 100k / 16.2k = on above 9 V." (exclude_from_sim no) (at 25.4 33.02 0) (effects (font (size 1.8 1.8)) (justify left)))
 (text "Output 4 x 47 uF 16 V + 220 uF polymer for servo stall pulses (8 A, 10 A peak)." (exclude_from_sim no) (at 25.4 38.1 0) (effects (font (size 1.8 1.8)) (justify left)))
