File: boards/drive/atlas_drive.kicad_pcb (KiCad board)
At the start: 6 copper layers, 140 x 90 mm, 408 parts, among them J1001 STACK_2x20, J101 B+, J102 B-, J103 PACK_SENSE, J401 BTN_EXT, J501 MOTOR A, J502 MOTOR B, J503 MOTOR C, J504 ESTOP, J601 SWD, J602 CAN, J603 HALL, J701 USB_C_16P, J702 EEPROM_PROG, J901 SERVO, J902 LIDAR_PWR, J903 FAN, Q201 CSD18510Q5B, Q202 CSD18510Q5B, Q203 CSD18510Q5B, Q204 CSD18510Q5B, Q205 CSD18510Q5B, Q206 CSD18510Q5B, Q207 CSD18510Q5B, Q208 CSD18510Q5B, Q301 MMBT3904, Q302 CSD18510Q5B, Q303 CSD18510Q5B, Q304 CSD18510Q5B, Q305 CSD18510Q5B, Q306 CSD18510Q5B, Q401 2N7002K, Q501 2N7002K, Q502 CSD18510Q5B, Q503 CSD18510Q5B, Q504 CSD18510Q5B, Q505 CSD18510Q5B, Q506 2N7002K, Q507 CSD18510Q5B, Q508 CSD18510Q5B, Q509 CSD18510Q5B, Q510 CSD18510Q5B, Q511 2N7002K, Q512 CSD18510Q5B, Q513 CSD18510Q5B, Q514 CSD18510Q5B, Q515 CSD18510Q5B, SW401 POWER, SW801 FLASH, U1001 INA228, U1002 24AA02, U201 BQ7791508, U301 TPS48111-Q1, U401 TPS70933, U402 SN74LVC1G74, U403 74LVC1G34, U404 TLV75533P, U501 DRV8323RS, U502 74LVC1G08, U601 STM32F405RGT6, U602 LSM6DS3TR-C, U603 SN65HVD230, U604 74AHCT1G125, U701 TPS25751D, U702 M24512, U703 BQ25798, U801 TS3USB30E, U802 TS3USB30E, U803 USB2514B, U804 CP2102N-QFN24, U901 TPSM63610, U902 TPS26600, Y601 8MHz, Y801 24MHz

Commit message: Add PCBWay silkscreen branding to both boards (Future Innovators Program requirement)
Drive: vertical 1.6 mm text at (45, 86) in the strip the brain board doesn't cover.
Brain: 2.0 mm text at (96, 57.25), above the 40-pin header, outside the Jetson module.
Both spots clear of pads, holes, vias, courtyards and other silkscreen.
Run DRC and regenerate fab files on the KiCad machine: run_kicad.sh drc-drive fab-drive drc-brain fab-brain

Co-Authored-By: Claude Opus 5.5 <noreply@anthropic.com>
Claude-Session: https://claude.ai/code/session_01TnZbLRjxD6Vfoy9VM5v47G
Other:
- board text added: "PCBWay"
Changed lines of the file:
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@@
+		)
+	)
+	(gr_text "PCBWay"
+		(at 45 86 90)
+		(layer "F.SilkS")
+		(effects
+			(font
+				(size 1.6 1.6)
+				(thickness 0.25)
+				(bold yes)
+			)
 		)
 	)
