File: boards/drive/atlas_drive.kicad_pcb (KiCad board)
At the start: 6 copper layers, 140 x 90 mm, 408 parts, among them J1001 STACK_2x20, J101 B+, J102 B-, J103 PACK_SENSE, J401 BTN_EXT, J501 MOTOR A, J502 MOTOR B, J503 MOTOR C, J504 ESTOP, J601 SWD, J602 CAN, J603 HALL, J701 USB_C_16P, J702 EEPROM_PROG, J901 SERVO, J902 LIDAR_PWR, J903 FAN, Q201 CSD18510Q5B, Q202 CSD18510Q5B, Q203 CSD18510Q5B, Q204 CSD18510Q5B, Q205 CSD18510Q5B, Q206 CSD18510Q5B, Q207 CSD18510Q5B, Q208 CSD18510Q5B, Q301 MMBT3904, Q302 CSD18510Q5B, Q303 CSD18510Q5B, Q304 CSD18510Q5B, Q305 CSD18510Q5B, Q306 CSD18510Q5B, Q401 2N7002K, Q501 2N7002K, Q502 CSD18510Q5B, Q503 CSD18510Q5B, Q504 CSD18510Q5B, Q505 CSD18510Q5B, Q506 2N7002K, Q507 CSD18510Q5B, Q508 CSD18510Q5B, Q509 CSD18510Q5B, Q510 CSD18510Q5B, Q511 2N7002K, Q512 CSD18510Q5B, Q513 CSD18510Q5B, Q514 CSD18510Q5B, Q515 CSD18510Q5B, SW401 POWER, SW801 FLASH, U1001 INA228, U1002 24AA02, U201 BQ7791508, U301 TPS48111-Q1, U401 TPS70933, U402 SN74LVC1G74, U403 74LVC1G34, U404 TLV75533P, U501 DRV8323RS, U502 74LVC1G08, U601 STM32F405RGT6, U602 LSM6DS3TR-C, U603 SN65HVD230, U604 74AHCT1G125, U701 TPS25751D, U702 M24512, U703 BQ25798, U801 TS3USB30E, U802 TS3USB30E, U803 USB2514B, U804 CP2102N-QFN24, U901 TPSM63610, U902 TPS26600, Y601 8MHz, Y801 24MHz

Commit message: Drive board: POWER_EN fix (R609 to +3V3, new R625 pull-down on GATE_EN_MCU)
Approved by Ragini, Sept 29.
- R609 (100k) now pulls STK_POWER_EN up to +3V3 instead of down to GND, so the brain board and
  the Jetson stay powered while the STM32 is in reset, being flashed, or blank.
- R625 (10k, 0402) pulls GATE_EN_MCU (PB5, U502 input A) down, so the gate driver stays off
  while the STM32 is in reset or in its ROM bootloader. Placed on the GATE_EN_MCU track next to
  U502 with its own GND via; placement recorded in out/atlas_drive_placement.json.
- Layout: R609's GND stub and via taken off. mazeroute.py routed R609 pad 2 to +3V3 (In2, two
  0.5 mm vias) and joined C619's ground (the piece of top pour that lost its via) to GND; for
  that it moved one stretch of the +3V3 trunk to B.Cu and part of TEMP_MOTOR. add_routes.py
  applied both.
- DRC: identical to Sept 27 (no unconnected items, no clearance errors, 0 schematic parity
  issues; the same 8 silkscreen/track-end warnings). ERC unchanged. Brain DRC unchanged (253,
  all inherited from Antmicro).
- Fab files for both boards regenerated with KiCad 10.0.6 (PCBWay logo now rendered by KiCad),
  and the top/bottom/iso renders.
- docs/FLASHING.md, docs/ARCHITECTURE.md: the fix is applied. atlas.conf now defaults to
  ATLAS_POWER_EN_FIXED=1; the atlas stm32 refusal message explains the flag.

Co-Authored-By: Claude Opus 5.5 <noreply@anthropic.com>
Claude-Session: https://claude.ai/code/session_01TnZbLRjxD6Vfoy9VM5v47G
Parts:
- added R625: 10k, Resistor_SMD:R_0402_1005Metric, F.Cu at (62.0, 107.8)
Connections:
- R609 pad 2: GND -> +3V3
Routing:
- net TEMP_MOTOR: track 22.8 -> 28.5 mm
- net GND: track 294.8 -> 298.4 mm
- net +3V3: track 707.9 -> 704.9 mm, vias 12 -> 14
