File: boards/drive/atlas_drive_f_mcu.kicad_sch (KiCad schematic)
At the start: 57 parts, among them J601 SWD, J602 CAN, J603 HALL, U601 STM32F405RGT6, U602 LSM6DS3TR-C, U603 SN65HVD230, U604 74AHCT1G125, Y601 8MHz

Commit message: Drive board: POWER_EN fix (R609 to +3V3, new R625 pull-down on GATE_EN_MCU)
Approved by Ragini, Sept 29.
- R609 (100k) now pulls STK_POWER_EN up to +3V3 instead of down to GND, so the brain board and
  the Jetson stay powered while the STM32 is in reset, being flashed, or blank.
- R625 (10k, 0402) pulls GATE_EN_MCU (PB5, U502 input A) down, so the gate driver stays off
  while the STM32 is in reset or in its ROM bootloader. Placed on the GATE_EN_MCU track next to
  U502 with its own GND via; placement recorded in out/atlas_drive_placement.json.
- Layout: R609's GND stub and via taken off. mazeroute.py routed R609 pad 2 to +3V3 (In2, two
  0.5 mm vias) and joined C619's ground (the piece of top pour that lost its via) to GND; for
  that it moved one stretch of the +3V3 trunk to B.Cu and part of TEMP_MOTOR. add_routes.py
  applied both.
- DRC: identical to Sept 27 (no unconnected items, no clearance errors, 0 schematic parity
  issues; the same 8 silkscreen/track-end warnings). ERC unchanged. Brain DRC unchanged (253,
  all inherited from Antmicro).
- Fab files for both boards regenerated with KiCad 10.0.6 (PCBWay logo now rendered by KiCad),
  and the top/bottom/iso renders.
- docs/FLASHING.md, docs/ARCHITECTURE.md: the fix is applied. atlas.conf now defaults to
  ATLAS_POWER_EN_FIXED=1; the atlas stm32 refusal message explains the flag.

Co-Authored-By: Claude Opus 5.5 <noreply@anthropic.com>
Claude-Session: https://claude.ai/code/session_01TnZbLRjxD6Vfoy9VM5v47G
Parts:
- added R625: 10k, Resistor_SMD:R_0402_1005Metric, symbol Device:R
Connections:
- net +3V3: now also R609.2
- net GATE_EN_MCU: now also R625.1
- net GND: now also R625.2; no longer R609.2
Other:
- moved on the sheet: C613, C614, C615, C616, C617, C618, C619, C620, D603, R610, R611, R612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
