File: boards/brain/atlas_brain.kicad_pcb (KiCad board)
At the start: 8 copper layers, 120 x 90 mm, 366 parts, among them J1 Bus_M.2_2199230-6, J10 Molex_PicoBlade_1x4_0533980471, J1001 STACK_2x20, J1301 LIDAR, J14 JST_SH_1x4_SM04B-SRSS-TB-LF-SN, J15 Bus_DDR4_SODIMM_CUSTOM_Jetson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, J2 Bus_M.2_1-2199230-6, J6 Bus_RJ45_5-2337992-8, M1 Jetson-Orin-NX-Nano, M3 Mech_M2_2280_H2.5mm, Q10 PJE138K, Q1001 SSM3J332R, Q1002 PJE138K, Q1003 PJE138K, Q1004 PJE138K, Q11 PJE138K, Q1201 CSD19538Q3A, Q1202 CSD19538Q3A, Q14 BCM857BS-7-F, Q16 SSM3J332R, Q18 SSM3J332R, Q22 PJE138K, Q5 PJE138K, Q6 SSM3J332R, Q7 PJE138K, Q8 PJE138K, Q9 PJE138K, SW1 SW_SPDT_PCM12SMTR, U1 SIC431AED-T1-GE3, U1001 NTS0102, U1101 TPS259474, U1201 LM5155, U1202 TPS23861, U1301 LAN7800, U2 74LVC2G07_SOT457, U29 TPS259474, U3 74LVC2G07_SOT457, U30 TPD4E05U06QDQARQ1, U33 NTS0102_XSON, U34 PCAL6408A_VQFN, U35 AP22653_DFN, U37 74LVC2G14_SOT457, U38 74LVC1G175_SOT457, U4 NTS0102_XSON, U40 SIC431AED-T1-GE3, U41 NCP730BMT330_WSON, U42 TPS7A0518P_SOT23-5, U48 TPS259474, Y1 Oscillator_32.768kHz_ECS_2520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, Y1301 25MHz

Commit message: Add PCBWay silkscreen branding to both boards (Future Innovators Program requirement)
Drive: vertical 1.6 mm text at (45, 86) in the strip the brain board doesn't cover.
Brain: 2.0 mm text at (96, 57.25), above the 40-pin header, outside the Jetson module.
Both spots clear of pads, holes, vias, courtyards and other silkscreen.
Run DRC and regenerate fab files on the KiCad machine: run_kicad.sh drc-drive fab-drive drc-brain fab-brain

Co-Authored-By: Claude Opus 5.5 <noreply@anthropic.com>
Claude-Session: https://claude.ai/code/session_01TnZbLRjxD6Vfoy9VM5v47G
Other:
- board text added: "PCBWay"
Changed lines of the file:
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@@
+		)
+	)
+	(gr_text "PCBWay"
+		(at 96 57.25)
+		(layer "F.SilkS")
+		(effects
+			(font
+				(size 2.0 2.0)
+				(thickness 0.3)
+				(bold yes)
+			)
 		)
 	)
