File: boards/power/atlas_power_a_pack.kicad_sch (KiCad schematic)
At the start: 9 parts, among them J101 BAT+, J102 BAT-

Commit message: Rev B: design fixes from the review (B1, M1, M2, M3, M6, M7, minors)
Charge ground split (CHG_GND, MOD502 OUT- the only tie to GND, netcheck rule
14); 1 k series into the dev kit's level-shifted inputs; IRF4905PBF with 6.8 k
dividers and gate caps on the dev-kit and charge P-FETs; BEC+ alternate pad on
VSYS_SW; series resistors on the FSESC signal grounds; through-hole USB-A for
the dev kit; R304 2.2 M, C1001 10 nF, P6KE22A on the dev-kit, lidar and camera
feeds, 10 k NTC series resistor, R408 4.7 ohm; DIP sockets in the BOM; XT90-S
gender stated. 215 parts, 133 nets, netcheck 0 errors, 49.37 per board.

Co-Authored-By: Claude Fable 5.1 <noreply@anthropic.com>
Claude-Session: https://claude.ai/code/session_01BogQQgJLXFQcAbYtKpDqRe
Other:
- note added: "Pack lead: 10 AWG pigtail soldered into J101/J102 with an XT90 male on its end. The pack carries the"
- note added: "XT90-S female: the anti-spark resistor sits in the female half (probots and myfpvstore listings; one"
- note added: "esk8.news teardown says male, so check with a meter: the half with a few ohms between two contacts of one"
- note added: "pole goes on the pack). Also on the pack: 125 A MIDI fuse at B+, JBD BMS in B-. P- after the BMS is board GND."
- note removed: "Pack lead: 10 AWG pigtail soldered into J101/J102 with an XT90 male on its end; the pack carries the"
- note removed: "XT90-S anti-spark female, the 125 A MIDI fuse at B+ and the JBD BMS in B-. P- after the BMS is board GND."
- moved on the sheet: C101, C102, C103, C104, D101, J101, J102, TP101, TP102
