File: boards/power/atlas_power_c_switch.kicad_sch (KiCad schematic)
At the start: 33 parts, among them Q301 IRFB7430PBF, Q302 IRFB7430PBF, Q303 IRFB7430PBF, Q304 IRF9Z34NPBF, Q305 2N3904, U301 MIC5014, U302 74HCT08

Commit message: Rev B: design fixes from the review (B1, M1, M2, M3, M6, M7, minors)
Charge ground split (CHG_GND, MOD502 OUT- the only tie to GND, netcheck rule
14); 1 k series into the dev kit's level-shifted inputs; IRF4905PBF with 6.8 k
dividers and gate caps on the dev-kit and charge P-FETs; BEC+ alternate pad on
VSYS_SW; series resistors on the FSESC signal grounds; through-hole USB-A for
the dev kit; R304 2.2 M, C1001 10 nF, P6KE22A on the dev-kit, lidar and camera
feeds, 10 k NTC series resistor, R408 4.7 ohm; DIP sockets in the BOM; XT90-S
gender stated. 215 parts, 133 nets, netcheck 0 errors, 49.37 per board.

Co-Authored-By: Claude Fable 5.1 <noreply@anthropic.com>
Claude-Session: https://claude.ai/code/session_01BogQQgJLXFQcAbYtKpDqRe
Parts:
- added R316: 10k, Resistor_SMD:R_1206_3216Metric_Pad1.30x1.75mm_HandSolder, symbol Device:R
- R304: value 100k -> 2.2M; MPN RC1206FR-07100KL -> RC1206FR-072M2L
Connections:
- net FET_NTC: now also R316.2; no longer R314.2, TH301.1
- new net NTC_NODE: R314.2, R316.1, TH301.1
Other:
- note added: "10 Ohm per gate (sharing, damping), 2.2M G-S keeps the FETs off with the MIC5014 out of its socket (100k"
- note added: "R313; at 4.7 Ohm the peak is 3.6 A for about 10 ms (check that the MF-R050 does not trip)."
- note added: "Review M3: the FSESC and the Castle BEC load VM during precharge (110 mA is the limit at 12 V). If the bench"
- note added: "loaded its charge pump, review m1)."
- note added: "test fails: move the BEC lead to J410 (VSYS_SW) and/or fit 4.7 Ohm 5 W (Yageo SQP500JB-4R7, same body) as"
- note removed: "10 Ohm per gate (sharing, damping), 100k G-S keeps the FETs off with the MIC5014 out of its socket."
- moved on the sheet: C301, C302, C303, C304, D301, D302, F301, HS301, Q301, Q302, Q303, Q304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
