File: boards/power/atlas_power_d_rails.kicad_sch (KiCad schematic)
At the start: 61 parts, among them J401 BEC+, J402 BEC-, J403 BEC_OUT, J404 SRV+, J405 SRV-, J406 SERVO, J407 DEV+, J408 DEV-, J409 LIDAR_PWR, Q401 2N3904, Q402 IRF9Z34NPBF, Q403 2N3904, Q404 2N3906, Q405 IRF9Z34NPBF, Q406 2N3904, SW401 POWER, U401 R-78E5.0-1.0, U402 TL431

Commit message: Rev B: design fixes from the review (B1, M1, M2, M3, M6, M7, minors)
Charge ground split (CHG_GND, MOD502 OUT- the only tie to GND, netcheck rule
14); 1 k series into the dev kit's level-shifted inputs; IRF4905PBF with 6.8 k
dividers and gate caps on the dev-kit and charge P-FETs; BEC+ alternate pad on
VSYS_SW; series resistors on the FSESC signal grounds; through-hole USB-A for
the dev kit; R304 2.2 M, C1001 10 nF, P6KE22A on the dev-kit, lidar and camera
feeds, 10 k NTC series resistor, R408 4.7 ohm; DIP sockets in the BOM; XT90-S
gender stated. 215 parts, 133 nets, netcheck 0 errors, 49.37 per board.

Co-Authored-By: Claude Fable 5.1 <noreply@anthropic.com>
Claude-Session: https://claude.ai/code/session_01BogQQgJLXFQcAbYtKpDqRe
Parts:
- added C407: 100n, Capacitor_SMD:C_1206_3216Metric_Pad1.33x1.80mm_HandSolder, symbol Device:C
- added D406: P6KE22A, Diode_THT:D_DO-15_P3.81mm_Vertical_KathodeUp, symbol Device:D_Zener
- added J410: BEC+ALT, Connector_Wire:SolderWire-1.5sqmm_1x01_D1.7mm_OD3.9mm, symbol atlas:PAD_BEC_IN+ALT
- D404, D405: value P6KE20A -> P6KE22A; MPN P6KE20A -> P6KE22A; Manufacturer Littelfuse -> Taiwan Semiconductor; Price 0.54 -> 0.45; Source https://www.findchips.com/search/P6KE20A -> https://www.findchips.com/search/P6KE22A
- Q402: value IRF9Z34NPBF -> IRF4905PBF; symbol atlas:IRF9Z34NPBF -> atlas:IRF4905PBF; MPN IRF9Z34NPBF -> IRF4905PBF; Price 1.08 -> 2.71; Source https://www.findchips.com/search/IRF9Z34NPBF -> https://www.findchips.com/search/IRF4905PBF
- R408: value 10 -> 4.7; MPN Vishay MBB02070C1009FCT00 (0.6 W metal film) -> Vishay MBB02070C4708FCT00 (0.6 W metal film); Price 0.24 -> 0.26; Source https://www.findchips.com/search/MBB02070C1009FCT00 -> https://www.findchips.com/search/MBB02070C4708FCT00
- R412: value 10k -> 6.8k; MPN RC1206FR-0710KL -> RC1206FR-076K8L
Connections:
- net CAM_VIN: now also D406.1 (K)
- net GND: now also D406.2 (A)
- net OV_G: now also C407.2
- net VDEV_F: now also C407.1
- net VSYS_SW: now also J410.1
Other:
- note added: "Camera: MF-R075 -> P6KE22A -> wire pads -> Pololu S18V20F12 (off board) -> camera lead."
- note added: "Dev kit: 5 A mini blade fuse -> P6KE22A -> over-voltage cut-off (IRF4905, TL431 trips at 18.7 V, releases 17.85 V)"
- note added: "Lidar: IRF9Z34N high side, 10k/10k gate divider, 100 nF soft start, MF-R075, P6KE22A, Phoenix 2-pin."
- note added: "R-78E5.0-1.0 (8-28 V in) behind 4.7 Ohm + P6KE20A, so a 30 V spike on VSYS_SW reaches it as <= 22 V."
- note added: "Servo: Castle BEC 2.0 from VM (J401), or from VSYS_SW (J410) if its start-up load stops the precharge (M3)."
- note removed: "Camera: MF-R075 -> wire pads -> Pololu S18V20F12 (off board) -> camera lead. Servo: Castle BEC 2.0 from VM."
- note removed: "Dev kit: 5 A mini blade fuse -> P6KE20A -> over-voltage cut-off (IRF9Z34N, TL431 trips at 18.6 V, releases 17.9 V)"
- note removed: "Lidar: IRF9Z34N high side, 10k/10k gate divider, 100 nF soft start, MF-R075, P6KE20A, Phoenix 2-pin."
- note removed: "R-78E5.0-1.0 (8-28 V in) behind 10 Ohm + P6KE20A, so a 30 V spike on VSYS_SW reaches it as <= 22 V."
- moved on the sheet: C401, C402, C403, C404, C405, C406, D401, D402, D403, D404, D405, F401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
