File: boards/power/atlas_power_e_charge.kicad_sch (KiCad schematic)
At the start: 17 parts, among them Q501 IRF9Z34NPBF, Q502 2N3904, Q503 2N3904

Commit message: Rev B: design fixes from the review (B1, M1, M2, M3, M6, M7, minors)
Charge ground split (CHG_GND, MOD502 OUT- the only tie to GND, netcheck rule
14); 1 k series into the dev kit's level-shifted inputs; IRF4905PBF with 6.8 k
dividers and gate caps on the dev-kit and charge P-FETs; BEC+ alternate pad on
VSYS_SW; series resistors on the FSESC signal grounds; through-hole USB-A for
the dev kit; R304 2.2 M, C1001 10 nF, P6KE22A on the dev-kit, lidar and camera
feeds, 10 k NTC series resistor, R408 4.7 ohm; DIP sockets in the BOM; XT90-S
gender stated. 215 parts, 133 nets, netcheck 0 errors, 49.37 per board.

Co-Authored-By: Claude Fable 5.1 <noreply@anthropic.com>
Claude-Session: https://claude.ai/code/session_01BogQQgJLXFQcAbYtKpDqRe
Parts:
- added C502: 100n, Capacitor_SMD:C_1206_3216Metric_Pad1.33x1.80mm_HandSolder, symbol Device:C
- added TP502: CHG_GND, TestPoint:TestPoint_THTPad_1.5x1.5mm_Drill0.7mm, symbol Connector:TestPoint
- Q501: value IRF9Z34NPBF -> IRF4905PBF; symbol atlas:IRF9Z34NPBF -> atlas:IRF4905PBF; MPN IRF9Z34NPBF -> IRF4905PBF; Price 1.08 -> 2.71; Source https://www.findchips.com/search/IRF9Z34NPBF -> https://www.findchips.com/search/IRF4905PBF
- R502: value 10k -> 6.8k; MPN RC1206FR-0710KL -> RC1206FR-076K8L
Connections:
- net CHG_G: now also C502.2
- net CHG_RB: now also C502.1
- net GND: no longer C501.2, D501.2 (A), MOD501.2 (GND), MOD502.2 (IN-), Q502.1 (E), Q503.1 (E), R504.2, R506.2
- new net CHG_GND: C501.2, D501.2 (A), MOD501.2 (GND), MOD502.2 (IN-), Q502.1 (E), Q503.1 (E), R504.2, R506.2, TP502.1
Other:
- note added: "Charge ground (review B1): the common XL4015 CC/CV module measures current with a shunt between IN- and"
- note added: "OUT-. So the charger side has its own net CHG_GND (PD trigger GND, CC/CV IN-, D501, C501, the charger-present"
- note added: "Reverse block: Q501 IRF4905 with its body diode toward the pack, turned fully on only while CHG_IN > ~17.5 V"
- note added: "detector) and CC/CV OUT- is its only tie to GND: the charge current returns through the shunt and CC works. A"
- note added: "module with high-side sensing (IN- and OUT- joined inside) works on the same pads. Bench check in README."
- note removed: "Reverse block: Q501 P-FET with its body diode toward the pack, turned fully on only while CHG_IN > ~17.5 V"
- moved on the sheet: C501, D501, D502, F501, MOD501, MOD502, Q501, Q502, Q503, R501, R502, R503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
