File: boards/power/atlas_power_f_debug.kicad_sch (KiCad schematic)
At the start: 13 parts, among them J601 DEVKIT_USB, J602 VESC_USB, J603 HUB_PORT4, U601 MCP2221A, U602 MCP1700-3302E/TO

Commit message: Rev B: design fixes from the review (B1, M1, M2, M3, M6, M7, minors)
Charge ground split (CHG_GND, MOD502 OUT- the only tie to GND, netcheck rule
14); 1 k series into the dev kit's level-shifted inputs; IRF4905PBF with 6.8 k
dividers and gate caps on the dev-kit and charge P-FETs; BEC+ alternate pad on
VSYS_SW; series resistors on the FSESC signal grounds; through-hole USB-A for
the dev kit; R304 2.2 M, C1001 10 nF, P6KE22A on the dev-kit, lidar and camera
feeds, 10 k NTC series resistor, R408 4.7 ohm; DIP sockets in the BOM; XT90-S
gender stated. 215 parts, 133 nets, netcheck 0 errors, 49.37 per board.

Co-Authored-By: Claude Fable 5.1 <noreply@anthropic.com>
Claude-Session: https://claude.ai/code/session_01BogQQgJLXFQcAbYtKpDqRe
Parts:
- added R604: 2.2, Resistor_SMD:R_1206_3216Metric_Pad1.30x1.75mm_HandSolder, symbol Device:R
- J601: footprint Connector_PinHeader_2.54mm:PinHeader_1x04_P2.54mm_Vertical -> Connector_USB:USB_A_Wuerth_614004134726_Horizontal; MPN Wurth 61300411121 -> Wurth 614004134726; Price 0.19 -> 3.87; Source https://www.findchips.com/search/61300411121 -> https://www.findchips.com/search/614004134726
- R602: value 10k -> 1k; MPN RC1206FR-0710KL -> RC1206FR-071KL
Connections:
- net GND: now also J601.5 (SHIELD), R604.2; no longer J602.4 (GND)
- new net VUSB_GND: J602.4 (GND), R604.1
Other:
- note added: "USB-C (192.168.55.1; for flashing NVIDIA documents a direct cable: laptop straight into the dev kit is the"
- note added: "cannot power the car. GND is common. Port 1 -> J601 USB-A receptacle -> one USB-A to C cable -> dev-kit"
- note added: "fallback). Port 3 -> J602 -> 4449 -> the FSESC micro-USB cable, its ground through 3.3 Ohm (M6)."
- note removed: "cannot power the car. GND is common. Port 1 -> J601 -> Adafruit 4449 jack lead -> USB-A to C cable ->"
- note removed: "dev-kit USB-C (192.168.55.1, flashing). Port 3 -> J602 -> 4449 -> the FSESC micro-USB cable."
- moved on the sheet: C601, C602, C603, C604, J602, J603, MOD601, R601, R602, R603, U601, U602
