File: boards/power/atlas_power_h_jetson.kicad_sch (KiCad schematic)
At the start: 22 parts, among them J801 J12_RIBBON, J802 J14_HARNESS, SW801 RECOVERY, U801 PC817, U802 PC817

Commit message: Rev B: design fixes from the review (B1, M1, M2, M3, M6, M7, minors)
Charge ground split (CHG_GND, MOD502 OUT- the only tie to GND, netcheck rule
14); 1 k series into the dev kit's level-shifted inputs; IRF4905PBF with 6.8 k
dividers and gate caps on the dev-kit and charge P-FETs; BEC+ alternate pad on
VSYS_SW; series resistors on the FSESC signal grounds; through-hole USB-A for
the dev kit; R304 2.2 M, C1001 10 nF, P6KE22A on the dev-kit, lidar and camera
feeds, 10 k NTC series resistor, R408 4.7 ohm; DIP sockets in the BOM; XT90-S
gender stated. 215 parts, 133 nets, netcheck 0 errors, 49.37 per board.

Co-Authored-By: Claude Fable 5.1 <noreply@anthropic.com>
Claude-Session: https://claude.ai/code/session_01BogQQgJLXFQcAbYtKpDqRe
Parts:
- R804, R812, R813: value 10k -> 1k; MPN RC1206FR-0710KL -> RC1206FR-071KL
Other:
- note added: "UART1 (pins 8 TX, 10 RX) passes to the FSESC COMM header, crossed (10k toward the FSESC, 1k toward the Jetson);"
- note added: "kit level-shifts these pins (TXB-type, holds a pin through about 4k), so 10k would not toggle them (review M1)."
- note added: "pin n to 41-n: nothing then shorts the dev-kit 5 V). Board outputs toward the Jetson are behind 1k: the dev"
- note added: "the VESC 3.3 V pin is not used."
- note removed: "UART1 (pins 8 TX, 10 RX) passes to the FSESC COMM header, crossed, 10k each way; the VESC 3.3 V pin is not used."
- note removed: "pin n to 41-n: nothing then shorts the dev-kit 5 V). Every board output toward the Jetson is behind 10k."
- moved on the sheet: J801, J802, R801, R802, R803, R804, R805, R806, R807, R808, R809, R810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
