File: boards/power/atlas_power_i_esc.kicad_sch (KiCad schematic)
At the start: 8 parts, among them J901 ESC+, J902 ESC-, J903 FSESC_COMM, J904 SERVO_IN

Commit message: Rev B: design fixes from the review (B1, M1, M2, M3, M6, M7, minors)
Charge ground split (CHG_GND, MOD502 OUT- the only tie to GND, netcheck rule
14); 1 k series into the dev kit's level-shifted inputs; IRF4905PBF with 6.8 k
dividers and gate caps on the dev-kit and charge P-FETs; BEC+ alternate pad on
VSYS_SW; series resistors on the FSESC signal grounds; through-hole USB-A for
the dev kit; R304 2.2 M, C1001 10 nF, P6KE22A on the dev-kit, lidar and camera
feeds, 10 k NTC series resistor, R408 4.7 ohm; DIP sockets in the BOM; XT90-S
gender stated. 215 parts, 133 nets, netcheck 0 errors, 49.37 per board.

Co-Authored-By: Claude Fable 5.1 <noreply@anthropic.com>
Claude-Session: https://claude.ai/code/session_01BogQQgJLXFQcAbYtKpDqRe
Parts:
- added R905, R906: 3.3, Resistor_SMD:R_1206_3216Metric_Pad1.30x1.75mm_HandSolder, symbol Device:R
Connections:
- net GND: now also R905.2, R906.2; no longer J903.2 (GND), J904.3 (GND)
- new net COMM_GND: J903.2 (GND), R905.1
- new net SRVIN_GND: J904.3 (GND), R906.1
Other:
- note added: "Review M6: the FSESC signal grounds (COMM pin 2, the servo lead, its USB) run beside its ESC- lead, which drops"
- note added: "about 90 mV at 90 A. Each goes to GND through 3.3 Ohm: 20-30 mA of loop current instead of amps, and the"
- note added: "resistor opens like a fuse if the ESC- joint fails. Run ESC+ and ESC- as one strain-relieved pair."
- moved on the sheet: J901, J902, J903, J904, R901, R902, R903, R904
