File: boards/power/atlas_power_j_misc.kicad_sch (KiCad schematic)
At the start: 20 parts, among them J1001 ESTOP, J1002 BTN_REMOTE, J1003 FAN, Q1001 2N7000

Commit message: Rev B: design fixes from the review (B1, M1, M2, M3, M6, M7, minors)
Charge ground split (CHG_GND, MOD502 OUT- the only tie to GND, netcheck rule
14); 1 k series into the dev kit's level-shifted inputs; IRF4905PBF with 6.8 k
dividers and gate caps on the dev-kit and charge P-FETs; BEC+ alternate pad on
VSYS_SW; series resistors on the FSESC signal grounds; through-hole USB-A for
the dev kit; R304 2.2 M, C1001 10 nF, P6KE22A on the dev-kit, lidar and camera
feeds, 10 k NTC series resistor, R408 4.7 ohm; DIP sockets in the BOM; XT90-S
gender stated. 215 parts, 133 nets, netcheck 0 errors, 49.37 per board.

Co-Authored-By: Claude Fable 5.1 <noreply@anthropic.com>
Claude-Session: https://claude.ai/code/session_01BogQQgJLXFQcAbYtKpDqRe
Parts:
- C1001: value 100n -> 10n; MPN Samsung CL31B104KBCNNNC (100 nF 50 V X7R 1206) -> KEMET C1206C103K5RACTU (10 nF 50 V X7R 1206); Manufacturer Samsung -> KEMET; Price 0.14 -> 0.10; Source https://www.findchips.com/search/CL31B104KBCNNNC -> https://www.findchips.com/search/C1206C103K5RACTU
Other:
- note added: "E-stop: 3.3 V -> 1k -> normally-closed loop (JST-PH 2) -> 100 Ohm -> ESTOP_OK, 10k + 10 nF to GND (0.1 ms;"
- note added: "review m3: a slow edge into the non-Schmitt 74HCT08 could chatter the main switch)."
- note removed: "E-stop: 3.3 V -> 1k -> normally-closed loop (JST-PH 2) -> 100 Ohm -> ESTOP_OK, 10k + 100 nF to GND."
- moved on the sheet: C1001, D1001, D1002, H1001, H1002, H1003, H1004, H1005, H1006, J1001, J1002, J1003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
