File: boards/power/atlas_power.kicad_pcb (KiCad board)
At the start: 2 copper layers, 130 x 84 mm, 218 parts, among them J1001 ESTOP, J1002 BTN_REMOTE, J1003 FAN, J101 BAT+, J102 BAT-, J201 BMS_UART, J401 BEC+, J402 BEC-, J403 BEC_OUT, J404 SRV+, J405 SRV-, J406 SERVO, J407 DEV+, J408 DEV-, J409 LIDAR_PWR, J410 BEC+ALT, J601 DEVKIT_USB, J602 VESC_USB, J603 HUB_PORT4, J801 J12_RIBBON, J802 J14_HARNESS, J901 ESC+, J902 ESC-, J903 FSESC_COMM, J904 SERVO_IN, Q1001 2N7000, Q301 IRFB7430PBF, Q302 IRFB7430PBF, Q303 IRFB7430PBF, Q304 IRF9Z34NPBF, Q305 2N3904, Q401 2N3904, Q402 IRF4905PBF, Q403 2N3904, Q404 2N3906, Q405 IRF9Z34NPBF, Q406 2N3904, Q501 IRF4905PBF, Q502 2N3904, Q503 2N3904, SW401 POWER, SW801 RECOVERY, U201 PC817, U202 PC817, U301 MIC5014, U302 74HCT08, U401 R-78E5.0-1.0, U402 TL431, U601 MCP2221A, U602 MCP1700-3302E/TO, U801 PC817, U802 PC817

Commit message: Rev B (WIP): ATLAS-PWR-1 routing, power paths done, 18 signal nets open
1869 tracks, 247 vias; BAT, VM, GND, VSYS_SW, servo and gate-drive paths
hand-routed and locked; mask openings over the BAT and VM pours; pour
resistance at 90 A: 1.035 mohm end to end (93 mV). 31 unconnected items remain
around the Pico / J802 header (placement fix pending). PCBWay instant quote
for 5 boards: $50.09 + $26.55 shipping. hand_routes.py and mazeroute options.

Co-Authored-By: Claude Fable 5.1 <noreply@anthropic.com>
Claude-Session: https://claude.ai/code/session_01BogQQgJLXFQcAbYtKpDqRe
Parts:
- moved TP403 94.8 mm to (74.0, 99.9)
- moved R401 61.0 mm to (106.5, 64.2)
- moved R701 50.8 mm to (100.0, 58.0), turned to -90 degrees
- moved C502 38.1 mm to (63.6, 91.5), turned to 90 degrees
- moved R811 18.9 mm to (90.0, 95.0)
- moved R813 16.1 mm to (71.8, 102.8), turned to 0 degrees
- moved R411 10.2 mm to (115.7, 59.6), turned to -90 degrees
- moved R306 3.15 mm to (92.0, 41.1)
- moved TP802 2.26 mm to (64.8, 99.5)
- moved R507 1.90 mm to (69.5, 98.5)
- moved C401 1.82 mm to (74.8, 94.8)
- moved J408 1.28 mm to (123.3, 45.8)
- moved R506 0.75 mm to (70.2, 92.8)
- moved R505 0.25 mm to (60.8, 86.8)
Routing:
- net SERVO_V: track 13.2 -> 173.7 mm, vias 0 -> 6
- net FAN_PWM: track 142.2 -> 0.00 mm, vias 2 -> 0
- net LIDAR_REQ: track 138.2 -> 0.00 mm, vias 2 -> 0
- net PICO_VSYS: track 4.47 -> 139.7 mm, vias 0 -> 6
- net JETSON_3V3_SENSE: track 133.3 -> 2.40 mm, vias 7 -> 0
- net I2C0_SDA: track 127.3 -> 0.00 mm, vias 3 -> 0
- net I2C0_SCL: track 125.3 -> 0.00 mm, vias 2 -> 0
- net VESC_KILL: track 120.6 -> 6.60 mm, vias 2 -> 0
- net +5V: track 213.8 -> 119.3 mm, vias 7 -> 1
- net ESTOP_OK_TO_JETSON: track 93.9 -> 0.00 mm
- net VSYS_SW: track 79.6 -> 142.3 mm, vias 1 -> 2
- net VDEV: track 0.00 -> 53.6 mm
- net CHG_RB: track 11.0 -> 62.0 mm, vias 0 -> 2
- net OV_C: track 45.7 -> 0.00 mm
- net BTN_HI: track 70.7 -> 115.6 mm, vias 2 -> 4
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
Commit message: Rev B: ATLAS-PWR-1 routed on 4 layers, DRC clean, PCBWay fab files
Two 2-layer attempts left 18-21 logic nets open around the Pico and the J14
header, so the board is now F.Cu 2 oz (parts, power pours), In1 solid GND
plane (BMS island cut out), In2 signals, B.Cu 2 oz. 1944 track segments,
435 vias (317 GND), 0 unconnected, 0 clearance errors. 90 A path 1.035 mohm
end to end; DEV- return 0.976 mohm. Gerbers (14 files), drill, PCBWay zip,
CPL, BOM and renders in boards/power/out. PCBWay instant quote, 5 pcs:
$155.79 + $26.55 shipping (2 oz outer / 1 oz inner).

Co-Authored-By: Claude Fable 5.1 <noreply@anthropic.com>
Claude-Session: https://claude.ai/code/session_01BogQQgJLXFQcAbYtKpDqRe
Parts:
- moved R801 102.9 mm to (130.2, 46.2), turned to 90 degrees
- moved R802 94.4 mm to (130.2, 51.5), turned to 90 degrees
- moved R813 92.4 mm to (157.8, 69.0), turned to 90 degrees
- moved R806 78.3 mm to (136.8, 73.5), turned to 90 degrees
- moved R807 73.1 mm to (139.5, 79.5), turned to 90 degrees
- moved R811 63.0 mm to (142.8, 60.5), turned to 90 degrees
- moved R812 61.4 mm to (142.8, 65.8)
- moved R809 60.5 mm to (130.2, 64.0), turned to 90 degrees
- moved C407 1.00 mm to (112.8, 64.5)
Routing:
- net FAN_PWM: track 0.00 -> 146.9 mm, vias 0 -> 1
- net CHG_STAT_N_TO_JETSON: track 133.2 -> 14.0 mm, vias 7 -> 0
- net VESC_KILL: track 6.60 -> 121.0 mm, vias 0 -> 1
- net J12_SCL: track 4.26 -> 118.6 mm, vias 0 -> 3
- net SERVO_IN_J: track 0.00 -> 113.2 mm, vias 0 -> 3
- net J12_SDA: track 3.35 -> 114.1 mm, vias 0 -> 2
- net J14_CON_RXD: track 0.00 -> 90.6 mm, vias 0 -> 4
- net J12_CHG_STAT_N: track 12.9 -> 97.7 mm, vias 0 -> 3
- net LATCH_OFF: track 0.00 -> 84.2 mm, vias 0 -> 3
- net J12_ESTOP_OK: track 14.3 -> 98.1 mm, vias 0 -> 5
- net J12_3V3: track 3.36 -> 86.7 mm, vias 0 -> 2
- net J12_LIDAR_REQ: track 21.5 -> 99.0 mm, vias 0 -> 5
- net +5V: track 119.3 -> 195.5 mm, vias 1 -> 0
- net JETSON_UP: track 77.6 -> 9.41 mm, vias 6 -> 0
- net PICO_VSYS: track 139.7 -> 91.6 mm, vias 6 -> 2
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- added copper zone on In1.Cu, net GND
Other:
- copper layers 2 -> 4
- board text added: "ATLAS-PWR-1 rev B 2026-10-26"
- board text removed: "ATLAS-PWR-1 rev B 2026-10-24"
